Commit message: Imported upstream version '0.0.28' of 'upstream'

File: robotino_description/urdf/arm.urdf.xacro (robot description, xacro)
@@ -166,5 +166,7 @@
       <type>transmission_interface/SimpleTransmission</type>
       <joint name="${name}base_joint">
+        <hardwareInterface>VelocityJointInterface</hardwareInterface>
         <hardwareInterface>PositionJointInterface</hardwareInterface>
+        <!--hardwareInterface>EffortJointInterface</hardwareInterface-->
       </joint>
       <actuator name="${name}base_motor">
@@ -177,5 +179,7 @@
       <type>transmission_interface/SimpleTransmission</type>
       <joint name="${name}joint${number}">
+        <hardwareInterface>VelocityJointInterface</hardwareInterface>
         <hardwareInterface>PositionJointInterface</hardwareInterface>
+        <!--hardwareInterface>EffortJointInterface</hardwareInterface-->
       </joint>
       <actuator name="arm_${number}_motor">

File: robotino_description/urdf/base.transmission.xacro (robot description, xacro)
@@ -18,7 +18,11 @@
       <joint name="${name}" >
         <hardwareInterface>VelocityJointInterface</hardwareInterface>
+        <hardwareInterface>PositionJointInterface</hardwareInterface>
+        <!--hardwareInterface>EffortJointInterface</hardwareInterface-->
       </joint>
       <actuator name="${name}_motor">
         <hardwareInterface>VelocityJointInterface</hardwareInterface>
+        <hardwareInterface>PositionJointInterface</hardwareInterface>
+        <!--hardwareInterface>EffortJointInterface</hardwareInterface-->
         <mechanicalReduction>${ 624/35 * 80/18}</mechanicalReduction>
       </actuator>

File: robotino_description/urdf/base.urdf.xacro (robot description, xacro)
@@ -102,5 +102,5 @@
       <origin xyz="0.01 0 0.12" rpy="0 0 0"/>
       <geometry>
-       <cylinder length="0.24" radius="0.23"/>
+       <mesh filename="package://robotino_description/meshes/RobotinoBody.stl"/>
       </geometry>
     </collision>
@@ -113,5 +113,5 @@
       <odometryFrame>odom</odometryFrame>
       <odometryRate>20.0</odometryRate>
-      <robotBaseFrame>origin</robotBaseFrame>
+      <robotBaseFrame>base_link</robotBaseFrame>
     </plugin>
   </gazebo>

Commit message: Rebase from 'upstream'

File: robotino_description/urdf/arm.urdf.xacro (robot description, xacro)
@@ -30,6 +30,6 @@
       <child link="${name}link1"/>
       <origin xyz="0.0 0.0 0.0" rpy="0 0 0" />
-      <axis xyz="0 1 0" />
-      <limit upper="1.5" lower="-1.2" effort="190" velocity="30" />
+      <axis xyz="0 -1 0" />
+      <limit upper="1.5" lower="-1.2" effort="90" velocity="0.7" />
     </joint>
     <link name="${name}link1">
@@ -57,5 +57,5 @@
       <origin xyz="0.0 0.0 0.25" rpy="0 0 0" />
       <axis xyz="0 1 0" />
-      <limit upper="2.3" lower="-1.7" effort="190" velocity="30" />
+      <limit upper="2.6" lower="-1.7" effort="90" velocity="0.7" />
     </joint>
     <link name="${name}motor2">
@@ -98,5 +98,5 @@
       <origin xyz="0.0 0.0 0.158" rpy="0 0 0" />
       <axis xyz="0 0 1" />
-      <limit upper="1.8" lower="-1.8" effort="190" velocity="30" />
+      <limit upper="1.8" lower="-1.8" effort="90" velocity="0.7" />
     </joint>
     <link name="${name}link3">
@@ -123,6 +123,6 @@
       <child link="${name}link4"/>
       <origin xyz="0.0 -0.057 0.065" rpy="0 0 0" />
-      <axis xyz="0 1 0" />
-      <limit upper="1.9" lower="-1.9" effort="160" velocity="30" />
+      <axis xyz="0 -1 0" />
+      <limit upper="2.4" lower="-2.4" effort="90" velocity="0.7" />
     </joint>
     <link name="${name}link4">
@@ -150,5 +150,5 @@
       <origin xyz="0.0 -0.027 0.035" rpy="0 0 0" />
       <axis xyz="0 0 1" />
-      <limit upper="2.9" lower="-2.9" effort="160" velocity="30" />
+      <limit upper="2.9" lower="-2.9" effort="90" velocity="0.7" />
     </joint>
     <link name="${name}link5">

File: robotino_description/urdf/base.gazebo.xacro (robot description, xacro)
@@ -6,4 +6,14 @@
   </xacro:macro>
   <xacro:macro name="base_gazebo" params="name">
+    <gazebo reference="origin">
+      <material>Gazebo/Grey</material>
+      <gravity>true</gravity>
+      <self_collide>false</self_collide>
+    </gazebo>
+    <gazebo reference="base_link">
+      <material>Gazebo/Grey</material>
+      <gravity>true</gravity>
+      <self_collide>false</self_collide>
+    </gazebo>
     <gazebo reference="${name}_linkx">
       <material>Gazebo/Grey</material>
@@ -17,9 +27,4 @@
     </gazebo>
     <gazebo reference="${name}_linkz">
-      <material>Gazebo/Grey</material>
-      <gravity>true</gravity>
-      <self_collide>false</self_collide>
-    </gazebo>
-    <gazebo reference="origin">
       <material>Gazebo/Grey</material>
       <gravity>true</gravity>

File: robotino_description/urdf/base.urdf.xacro (robot description, xacro)
@@ -20,4 +20,5 @@
     <limit upper="20" lower="-20" effort="190" velocity="30" />
    </joint>
+   <joints_transmission name="origin_joint" />
    <link name="${name}_link">
     <inertial>
@@ -34,5 +35,5 @@
     <origin xyz="0 0 0" rpy="0 0 0" />
     <axis xyz="1 0 0" />
-    <limit upper="20" lower="-20" effort="0" velocity="0" />
+    <limit upper="20" lower="-20" effort="90" velocity="0.3" />
     <dynamics damping="1000.0" friction="1000.0"/>
     <safety_controller k_velocity="10" k_position="15" soft_lower_limit="-10.0" soft_upper_limit="10.0" />
@@ -44,5 +45,5 @@
     <origin xyz="0 0 0" rpy="0 0 0" />
     <axis xyz="0 1 0" />
-    <limit upper="20" lower="-20" effort="0" velocity="0" />
+    <limit upper="20" lower="-20" effort="90" velocity="0.3" />
     <dynamics damping="1000.0" friction="1000.0"/>
     <safety_controller k_velocity="10" k_position="15" soft_lower_limit="-10.0" soft_upper_limit="10.0" />
@@ -54,5 +55,5 @@
     <origin xyz="0 0 0" rpy="0 0 0" />
     <axis xyz="0 0 1" />
-    <limit upper="3.14" lower="-3.14" effort="0" velocity="0" />
+    <limit upper="3.14" lower="-3.14" effort="90" velocity="0.7" />
     <dynamics damping="1000.0" friction="1000.0"/>
     <safety_controller k_velocity="10" k_position="15" soft_lower_limit="-3.14" soft_upper_limit="3.14" />
@@ -100,5 +101,5 @@
     </visual>
     <collision>
-      <origin xyz="0.01 0 0.12" rpy="0 0 0"/>
+      <origin xyz="0.01 0 0" rpy="0 0 0"/>
       <geometry>
        <mesh filename="package://robotino_description/meshes/RobotinoBody.stl"/>
@@ -113,5 +114,5 @@
       <odometryFrame>odom</odometryFrame>
       <odometryRate>20.0</odometryRate>
-      <robotBaseFrame>base_link</robotBaseFrame>
+      <robotBaseFrame>origin</robotBaseFrame>
     </plugin>
   </gazebo>

File: robotino_description/urdf/base_shell.urdf.xacro (robot description, xacro)
@@ -25,5 +25,5 @@
       </visual>
       <collision>
-        <origin xyz="0 0 0.05" rpy="0 0 -0.7"/>
+        <origin xyz="0 0 0.17" rpy="0 0 -0.7"/>
         <geometry>
           <mesh filename="package://robotino_description/meshes/base_shell_collision.stl"/>

File: robotino_description/urdf/hokuyo.urdf.xacro (robot description, xacro)
@@ -22,7 +22,7 @@
       </visual>
       <collision>
-        <origin xyz="0 0 ${HOKUYO_LENGTH/2}" rpy="0 0 0" />
+        <origin xyz="0 0 -0.035" rpy="0 0 0" />
         <geometry>
-          <cylinder radius="${HOKUYO_RADIUS}" length="${HOKUYO_LENGTH}" />
+          <cylinder radius="0.03" length="0.07" />
         </geometry>
       </collision>

File: robotino_description/urdf/shell.urdf.xacro (robot description, xacro)
@@ -2,5 +2,5 @@
 <root xmlns:xacro="http://www.ros.org/wiki/xacro">
   <xacro:include filename="$(find robotino_description)/urdf/kinect.urdf.xacro" />
-  <xacro:macro name="shell" params="name parent *origin">
+  <xacro:macro name="shell" params="name base_neck_x base_neck_y base_neck_z base_neck_roll base_neck_pitch base_neck_yaw parent *origin">
     <joint name="${name}_base_joint" type="fixed">
       <parent link="${parent}"/>
@@ -24,5 +24,5 @@
       </visual>
       <collision>
-        <origin xyz="0 0 0.05" rpy="0 0 -0.7"/>
+        <origin xyz="0 0 0" rpy="0 0 0"/>
         <geometry>
           <mesh filename="package://robotino_description/meshes/base_shell_collision.stl"/>
@@ -30,14 +30,41 @@
       </collision>
     </link>
-    <gazebo reference="${name}_link">
+    <gazebo reference="${name}_base_link">
       <gravity>true</gravity>
       <self_collide>false</self_collide>
       <material>Gazebo/LightGrey</material>
     </gazebo>
+    <joint name="base_neck_joint" type="fixed">
+      <origin xyz="${base_neck_x} ${base_neck_y} ${base_neck_z}" rpy="${base_neck_roll} ${base_neck_pitch} ${base_neck_yaw}"/>
+      <parent link="${parent}"/>
+      <child link="base_neck_link" />
+    </joint>
+   <link name="base_neck_link">
+      <inertial>
+        <mass value="0.00001" />
+        <origin xyz="0 0 0" />
+        <inertia ixx="1.0" ixy="0.0" ixz="0.0"
+          iyy="1.0" iyz="0.0"
+          izz="1.0" />
+      </inertial>
+      <visual>
+        <origin xyz="0 0 0" rpy="0 0 0" />
+        <geometry>
+          <box size="0.001 0.001 0.001" />
+        </geometry>
+        <material name="Black"/>
+      </visual>
+      <collision>
+        <origin xyz="0 0 0" rpy="0 0 0" />
+        <geometry>
+          <box size="0.001 0.001 0.001" />
+        </geometry>
+      </collision>
+    </link>
     <joint name="neck_pan_joint" type="revolute">
-      <origin xyz="0 0 0.676" rpy="0 0 0"/>
-      <parent link="${parent}"/>
+      <origin xyz="0 0 0" rpy="0 0 0"/>
+      <parent link="base_neck_link"/>
       <child link="neck_pan_link" />
-      <axis xyz="0 0 1" />
+      <axis xyz="0 0 -1" />
       <calibration rising="0.1"/>
       <limit effort="100" lower="-3.14" upper="3.14" velocity="1.4"/>
@@ -61,5 +88,5 @@
         <origin xyz="0 0 0" rpy="0 0 0"/>
         <geometry>
-          <mesh filename="package://robotino_description/meshes/neck.stl"/>
+          <cylinder length="0.08" radius="0.2"/>
         </geometry>
       </collision>
@@ -84,5 +111,5 @@
       <parent link="${parent}"/>
       <child link="head_link" />
-      <axis xyz="0 0 1" />
+      <axis xyz="0 0 -1" />
       <calibration rising="0.1"/>
       <limit effort="100" lower="-3.14" upper="3.14" velocity="1.4"/>
@@ -104,10 +131,66 @@
       </visual>
       <collision>
-        <origin xyz="0 0 0" rpy="0 0 0"/>
+        <origin xyz="0 0 0.125" rpy="0 0 0"/>
         <geometry>
-          <mesh filename="package://robotino_description/meshes/head.stl"/>
+          <cylinder length="0.25" radius="0.23"/>
         </geometry>
       </collision>
     </link>
+    <joint name="door_joint" type="revolute">
+      <origin xyz="0 0 0" rpy="0 0 0"/>
+      <parent link="${parent}"/>
+      <child link="door_link" />
+      <axis xyz="0 0 1" />
+      <calibration rising="0.1"/>
+      <limit effort="100" lower="0" upper="3.14" velocity="1.4"/>
+    </joint>
+   <link name="door_link">
+      <inertial>
+        <mass value="0.01"/>
+        <origin xyz="0 0 0"/>
+        <inertia ixx="0.001" ixy="0.0" ixz="0.0" iyy="0.001" iyz="0.0" izz="0.001" />
+      </inertial>
+      <visual>
+        <origin xyz="0 0 0" rpy="0 0 0"/>
+        <geometry>
+          <mesh filename="package://robotino_description/meshes/door.stl"/>
+        </geometry>
+        <material name="lightGrey">
+          <color rgba="0.9 0.9 0.9 1"/>
+        </material>
+      </visual>
+      <collision>
+        <origin xyz="0 0 0" rpy="0 0 0"/>
+        <geometry>
+          <mesh filename="package://robotino_description/meshes/door_collision.stl"/>
+        </geometry>
+      </collision>
+    </link>
+    <xacro:shell_transmission name="neck_pan"/>
+    <xacro:shell_transmission name="neck_tilt"/>
+    <xacro:shell_transmission name="head"/>
+    <xacro:shell_transmission name="door"/>
+    <xacro:shell_gazebo name="neck_base"/>
+    <xacro:shell_gazebo name="neck_pan"/>
+    <xacro:shell_gazebo name="neck_tilt"/>
+    <xacro:shell_gazebo name="head"/>
+    <xacro:shell_gazebo name="door"/>
+  </xacro:macro>
+  <xacro:macro name="shell_transmission" params="name">
+    <transmission name="${name}_joint_trans">
+      <type>transmission_interface/SimpleTransmission</type>
+      <joint name="${name}_joint">
+        <hardwareInterface>PositionJointInterface</hardwareInterface>
+      </joint>
+      <actuator name="${name}_joint_motor">
+        <mechanicalReduction>1</mechanicalReduction>
+      </actuator>
+    </transmission>
+  </xacro:macro>
+  <xacro:macro name="shell_gazebo" params="name">
+    <gazebo reference="${name}_link">
+      <gravity>true</gravity>
+      <self_collide>false</self_collide>
+    </gazebo>
   </xacro:macro>
 </root>
